File: sumo.kicad_sch (KiCad schematic)
At the start: 3 parts, among them U1 PIC16F628A-ISO

Commit message: recreate schematic
Parts:
- removed U1: PIC16F628A-ISO, symbol MCU_Microchip_PIC16:PIC16F628A-ISO
- added BT2: 9V, symbol Device:Battery
- added BT3: 6xAA, symbol Device:Battery
- added C1, C2: 1000uF, symbol Device:C_Polarized_US
- added C4: 1nF, symbol Device:C
- added C5, C8: 0.1uF, symbol Device:C
- added C6, C7: 1uF, symbol Device:C_Polarized_US
- added D1, D5: Super LED, symbol Device:LED
- added D2, D6: LED, symbol Device:LED
- added D3, D4: IR LED, LED_THT:LED_D3.0mm_IRBlack, symbol LED:IR204A
- added Q1, Q2: BPW40, LED_THT:LED_D5.0mm_Clear, symbol Sensor_Optical:BPW40
- added R1: 4.7k, symbol Device:R_US
- added R10, R15, R18, R6: 100, symbol Device:R_US
- added R11, R12, R16, R17: 220, symbol Device:R_US
- added R13, R4, R8: 230, symbol Device:R_US
- added R14, R5: 47k, symbol Device:R_US
- added R2, R3: 10k, symbol Device:R_US
- added R7: 100k, symbol Device:R_US
- added R9: 3.3k, symbol Device:R_US
- added SW1: SW_Push, symbol Switch:SW_Push
- added SW2: SW_DIP_x01, symbol Switch:SW_DIP_x01
- added T1, T2, T3, T4, T5: Screw_Terminal_01x04, symbol Connector:Screw_Terminal_01x04
- added U1: PIC16F628A-IP, symbol MCU_Microchip_PIC16:PIC16F628A-IP
- added U2: L7805, symbol Regulator_Linear:L7805
- added U3: L293D, Package_DIP:DIP-16_W7.62mm, symbol Driver_Motor:L293D
- added U4: 74HC04, symbol 74xx:74HC04
- added U5, U6: TSOP4038, OptoDevice:Vishay_MOLD-3Pin, symbol Interface_Optical:TSOP41xx
- added VR: 10k, symbol Device:R_Variable_US
- renumbered C1 to C3
Connections:
- net +6V: now also C6.1, C7.1, R10.2, R11.1, R13.1, R14.1, R17.1, R18.2, R4.1, R5.1, U4.12, U4.14 (VCC)
- net GNDREF: now also BT2.2 (-), C1.2, C5.1, C8.1, D1.1 (K), D5.1 (K), Q1.2 (E), Q2.2 (E), SW1.1, U1.5 (VSS), U2.2 (GND), U3.12 (GND), U3.13 (GND), U3.4 (GND), U3.5 (GND), U4.7 (GND), U5.2 (GND), U6.2 (GND)
- new net: R9.1, VR.1
- new net: U4.2, U4.3, VR.2
- new net: D6.2 (A), R17.2
- new net: R2.1, U3.1 (EN1,2)
- new net: T4.4 (Pin_4), U3.10 (3A)
- new net: T4.3 (Pin_3), U3.11 (3Y)
- new net: T4.2 (Pin_2), U3.14 (4Y)
- new net: T4.1 (Pin_1), U3.15 (4A)
- new net: R2.2, R3.1, SW2.2, U3.16 (VCC1), U3.8 (VCC2)
- new net: T3.1 (Pin_1), U3.2 (1A)
- new net: T3.2 (Pin_2), U3.3 (1Y)
- new net: T3.3 (Pin_3), U3.6 (2Y)
- new net: T3.4 (Pin_4), U3.7 (2A)
- new net: R3.2, U3.9 (EN3,4)
- new net: R8.2, U4.13
- new net: R7.2, U4.1
- new net: D1.2 (A), R4.2
- new net: Q2.1 (C), R14.2, R15.2
- new net: D3.1 (K), D4.1 (K), R8.1
- new net: T1.1 (Pin_1), U1.6 (RB0/INT)
- new net: T1.2 (Pin_2), U1.7 (RB1/RX/DT)
- new net: T1.3 (Pin_3), U1.8 (RB2/TX/CK)
- new net: T1.4 (Pin_4), U1.9 (RB3/CCP1)
- new net: C6.2, D2.1 (K), R12.1, U5.1 (OUT)
- new net: C5.2, R10.1, U5.3 (Vs)
- new net: R15.1, T5.2 (Pin_2)
- new net: C4.1, R7.1, R9.2
- new net: Q1.1 (C), R5.2, R6.2
- new net: R12.2, T5.3 (Pin_3)
- new net: C7.2, D6.1 (K), R16.1, U6.1 (OUT)
- new net: T2.2 (Pin_2), U1.1 (Vref/AN2/RA2)
- new net: T2.4 (Pin_4), U1.17 (AN0/RA0)
- new net: T2.3 (Pin_3), U1.18 (AN1/RA1)
- new net: T2.1 (Pin_1), U1.2 (CMP1/AN3/RA3)
- new net: R1.2, SW1.2, U1.4 (~{MCLR}/Vpp/RA5)
- new net: C8.2, R18.1, U6.3 (Vs)
- new net: BT3.1 (+), C2.1, SW2.1
- new net: BT3.2 (-), C2.2
- new net: R16.2, T5.4 (Pin_4)
- new net: D5.2 (A), R13.2
- new net: BT2.1 (+), U2.1 (IN)
- new net: R6.1, T5.1 (Pin_1)
- new net: D2.2 (A), R11.2
- new net: C4.2, U4.4, U4.5
- new net: D3.2 (A), D4.2 (A), U4.6
- new net +5V: C1.1, R1.1, U1.14 (VDD), U2.3 (OUT)
- no-connect marks 0 -> 6
Other:
- note added: "bot detection emitter"
- note added: "bot receier"
- note added: "line detector"
- note added: "motherboard"
- note added: "motor driver"
- note added: "webb's schematic says 12->13??"
- moved on the sheet: BT1, C3
